File: kicad/SchineLab_CoilFET_Board/SchineLab_CoilFET_Board.kicad_pcb (KiCad board)
At the start: 2 copper layers, 200 x 127 mm, 13 parts, among them J3 SENSE, J4 N-MOS, J8 P-MOS, J9 2491920000, Q1 Q_NMOS_GDS, Q2 Q_PMOS_GDS

Commit message: Updtate rear/FET board and added other files
Parts:
- added H1: MountingHole, MountingHole:MountingHole_4mm, F.Cu at (40.0, 36.4)
- added H2: MountingHole, MountingHole:MountingHole_4mm, F.Cu at (220.0, 36.4)
- added H3: MountingHole, MountingHole:MountingHole_4mm, F.Cu at (40.0, 150.7)
- added H4: MountingHole, MountingHole:MountingHole_4mm, F.Cu at (220.0, 150.7)
- moved C3 8.59 mm to (91.6, 60.0), turned to 180 degrees
- moved C4 6.84 mm to (84.7, 94.8), turned to 0 degrees
- moved C2 1.00 mm to (122.0, 116.0)
Routing:
- net -HCC: track 64.5 -> 0.00 mm
- net +HCC: track 69.4 -> 5.52 mm
- net GND: track 14.2 -> 17.5 mm, vias 6 -> 14
