File: kicad/SchineLab_CoilFET_Board/SchineLab_CoilFET_Board.kicad_sch (KiCad schematic)
At the start: 13 parts, among them J3 SENSE, J4 N-MOS, J8 P-MOS, J9 2491920000, Q1 Q_NMOS_GDS, Q2 Q_PMOS_GDS

Commit message: Updtate rear/FET board and added other files
Parts:
- added H1, H2, H3, H4: MountingHole, MountingHole:MountingHole_4mm, symbol Mechanical:MountingHole
Changed lines of the file:
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@@
+    )
+  )
+  (symbol (lib_id "Mechanical:MountingHole") (at 251.46 50.8 0) (unit 1)
+    (in_bom yes) (on_board yes) (dnp no) (fields_autoplaced)
+    (property "Reference" "H3" (at 254 49.53 0)
+      (effects (font (size 1.27 1.27)) (justify left))
+    )
+    (property "Value" "MountingHole" (at 254 52.07 0)
+      (effects (font (size 1.27 1.27)) (justify left))
+    )
+    (property "Footprint" "MountingHole:MountingHole_4mm" (at 251.46 50.8 0)
+      (effects (font (size 1.27 1.27)) hide)
+    )
+    (property "Datasheet" "~" (at 251.46 50.8 0)
+      (effects (font (size 1.27 1.27)) hide)
+    )
+    (instances
+      (project "SchineLab_CoilFET_Board"
+        (path "/2f21daab-ac04-42a8-876c-c86138d20a60"
+          (reference "H3") (unit 1)
+        )
+      )
     )
   )
@@
         )
       )
+    )
+  )
+  (symbol (lib_id "Mechanical:MountingHole") (at 251.46 41.91 0) (unit 1)
+    (in_bom yes) (on_board yes) (dnp no) (fields_autoplaced)
+    (property "Reference" "H2" (at 254 40.64 0)
+      (effects (font (size 1.27 1.27)) (justify left))
+    )
+    (property "Value" "MountingHole" (at 254 43.18 0)
+      (effects (font (size 1.27 1.27)) (justify left))
+    )
+    (property "Footprint" "MountingHole:MountingHole_4mm" (at 251.46 41.91 0)
+      (effects (font (size 1.27 1.27)) hide)
+    )
+    (property "Datasheet" "~" (at 251.46 41.91 0)
+      (effects (font (size 1.27 1.27)) hide)
+    )
+    (instances
+      (project "SchineLab_CoilFET_Board"
+        (path "/2f21daab-ac04-42a8-876c-c86138d20a60"
+          (reference "H2") (unit 1)
+        )
+      )
+    )
+  )
+  (symbol (lib_id "Mechanical:MountingHole") (at 251.46 59.69 0) (unit 1)
+    (in_bom yes) (on_board yes) (dnp no) (fields_autoplaced)
+    (property "Reference" "H4" (at 254 58.42 0)
+      (effects (font (size 1.27 1.27)) (justify left))
+    )
+    (property "Value" "MountingHole" (at 254 60.96 0)
+      (effects (font (size 1.27 1.27)) (justify left))
+    )
+    (property "Footprint" "MountingHole:MountingHole_4mm" (at 251.46 59.69 0)
+      (effects (font (size 1.27 1.27)) hide)
+    )
+    (property "Datasheet" "~" (at 251.46 59.69 0)
+      (effects (font (size 1.27 1.27)) hide)
+    )
+    (instances
+      (project "SchineLab_CoilFET_Board"
+        (path "/2f21daab-ac04-42a8-876c-c86138d20a60"
+          (reference "H4") (unit 1)
+        )
+      )
+    )
+  )
+  (symbol (lib_id "Mechanical:MountingHole") (at 251.46 33.02 0) (unit 1)
+    (in_bom yes) (on_board yes) (dnp no) (fields_autoplaced)
+    (property "Reference" "H1" (at 254 31.75 0)
+      (effects (font (size 1.27 1.27)) (justify left))
+    )
+    (property "Value" "MountingHole" (at 254 34.29 0)
+      (effects (font (size 1.27 1.27)) (justify left))
+    )
+    (property "Footprint" "MountingHole:MountingHole_4mm" (at 251.46 33.02 0)
+      (effects (font (size 1.27 1.27)) hide)
+    )
+    (property "Datasheet" "~" (at 251.46 33.02 0)
+      (effects (font (size 1.27 1.27)) hide)
+    )
+    (instances
+      (project "SchineLab_CoilFET_Board"
+        (path "/2f21daab-ac04-42a8-876c-c86138d20a60"
+          (reference "H1") (unit 1)
+        )
+      )
