File: kicad/H-bridge/H_bridge.kicad_sch (KiCad schematic)
At the start: 31 parts, among them J1 Screw_Terminal_01x02, J2 Conn_Coaxial, Q1 IAUT300N10S5N014ATMA1, Q2 IAUT300N10S5N014ATMA1, Q3 IAUT300N10S5N014ATMA1, Q4 IAUT300N10S5N014ATMA1, U1 LTV-817, U2 PDS1-S15-S15-M, U3 HIP4080A

Commit message: A few small adjustments
Parts:
- removed C3, C7, C8: C_Polarized, symbol Device:C_Polarized
- removed L6: LOAD, Inductors_SMD:L_0805, symbol Coil_speedifier-rescue:INDUCTOR-pspice
- added C3, C4, C7, C8, C9: C, symbol Device:C
- added J3: Loop_terminals, symbol Connector:Screw_Terminal_01x02
- added J4: Coil_terminals, symbol Connector:Screw_Terminal_01x02
Connections:
- net +15V: now also D1.2 (A), D2.2 (A), R5.1, U3.15 (VCC), U3.16 (VDD), C9.1
- net GNDD: now also R6.2, U3.3 (DIS), C4.2, C9.2, J3.2 (Pin_2)
- net at R2.1, R7.1, U1.3: now also C8.1
- net at Q3.3 (S), Q4.1 (D), U3.12 (AHS): now also C3.2, J4.2 (Pin_2)
- net at D1.1 (K), U3.1 (BHB): now also C7.1
- net at Q1.3 (S), Q2.1 (D), U3.19 (BHS): now also C7.2, J4.1 (Pin_1)
- net at Q1.1 (D), Q3.1 (D): now also J3.1 (Pin_1)
- net at D2.1 (K), U3.10 (AHB): now also C3.1
- net at R6.1: now also R5.2, U3.7 (IN-), C4.1
- net at U3.6 (IN+): now also R7.2, C8.2; no longer R6.2
Other:
- note added: "This box will contain the logic that will decide when it is safe to switch"
- moved on the sheet: J2, R1, R2, R5, R7, U1
