File: kicad/Controller_supply/Controller_supply.kicad_sch (KiCad schematic)
At the start: 10 parts, among them J1 Conn_01x03_Pin, J2 Conn_01x06_Pin, J3 Conn_01x04_Pin, U1 MC7824, U2 MC7924

Commit message: Updated internal power supply board and rear board.Please
Parts:
- added C5: 220uF, Capacitor_SMD:CP_Elec_10x10.5, symbol Device:C_Polarized_Small
- added J4: Conn_01x02, Connector_THT:Generic_7x7.5mm-footprt_1x02_P3.50mm_Horizontal, symbol Connector_Generic:Conn_01x02
- added U3: MC7824, Package_TO_SOT_SMD:TO-263-2, symbol Regulator_Linear:L7824
- D1: value CDBHD1100L-G -> GBU4A; footprint Package_TO_SOT_SMD:TO-269AA -> Diode_THT:Diode_Bridge_Vishay_GBU; symbol Diode_Bridge:ABS2 -> Diode_Bridge:GBU4A; DIGIKEY PARTNO 641-1209-1-ND -> GBU4A-ND; MPN CDBHD1100L-G -> GBU4A
- J1: footprint Connector_THT:CONN_1985205 -> Connector_THT:Generic_10.5x7.5mm-footprt_1x03_P3.50mm_Horizontal
- J3: footprint (none) -> Connector_THT:Generic_pin-to-housing_1x04_P5.00mm_Horizontal
Connections:
- net +24AC: now also D1.3; no longer D1.4
- net +24VDC: now also J1.1 (Pin_1)
- net -24AC: now also D1.2; no longer D1.3
- net -24VDC: now also J1.3 (Pin_3)
- net GND: now also C5.2, J4.2 (Pin_2), U3.2 (GND)
- net Line Hot: no longer J1.1 (Pin_1)
- net Line Neutral: no longer J1.3 (Pin_3)
- net at C1.1, D1.1 (+), U1.1 (IN): now also U3.1 (IN)
- net at C2.2, U2.2 (VI): now also D1.4 (-); no longer D1.2 (-)
- new net +24VDC_fan: C5.1, J4.1 (Pin_1), U3.3 (OUT)
